Commit message: updated wheel urdf

File: urdf/wheel.urdf.xacro (robot description, xacro)
@@ -3,6 +3,4 @@
   <!-- Properties -->
   <xacro:property name="PI" value="3.1415926535897931"/>
-  <!-- Base footprint -->
-  <link name="base_footprint"/>
   <!-- Robot base link with mesh -->
   <link name="base_link">
@@ -17,10 +15,4 @@
     </visual>
   </link>
-  <!-- Base footprint to base link joint -->
-  <joint name="base_footprint_to_base_link" type="fixed">
-    <parent link="base_footprint"/>
-    <child link="base_link"/>
-    <origin xyz="0.129 0 0.055" rpy="0 0 0"/>
-  </joint>
   <!-- Left wheel link -->
   <link name="left_wheel">

Commit message: Updated joy config and wheel diameter in control.h and base widh in urdf

File: urdf/wheel.urdf.xacro (robot description, xacro)
@@ -31,5 +31,5 @@
     <parent link="base_link"/>
     <child link="left_wheel"/>
-    <origin xyz="0.0 0.195 0" rpy="${-PI/2} 0 0"/>
+    <origin xyz="0.0 0.185 0" rpy="${-PI/2} 0 0"/>
     <axis xyz="0 0 1"/>
   </joint>
@@ -50,5 +50,5 @@
     <parent link="base_link"/>
     <child link="right_wheel"/>
-    <origin xyz="0.0 -0.195 0" rpy="${-PI/2} 0 0"/>
+    <origin xyz="0.0 -0.185 0" rpy="${-PI/2} 0 0"/>
     <axis xyz="0 0 1"/>
   </joint>
