Commit message: Humble code

File: urdf/uiabot.urdf.xacro (robot description, xacro)
@@ -6,5 +6,5 @@
   <link name="base_link">
     <visual>
-      <origin xyz="0.0 0.0 0.0" rpy="0 0 ${-pi/2}" />
+      <origin xyz="0.0 0.0 0.0" rpy="0 0 ${-PI/2}" />
       <geometry>
         <mesh scale="1 1 1" filename="package://uiabot/urdf/meshes/uiabot.stl"/>

Commit message: Update SAKO summerjob

File: urdf/uiabot.urdf.xacro (robot description, xacro)
@@ -33,5 +33,5 @@
   <link name="left_wheel">
     <visual>
-      <origin xyz="0 0 0" rpy="0 ${pi/2} 0" />
+      <origin xyz="0 0 0" rpy="0 ${PI/2} 0" />
       <geometry>
         <mesh scale="1 1 1" filename="package://uiabot/urdf/meshes/wheel.stl"/>
@@ -53,5 +53,5 @@
     <parent link="base_link"/>
     <child link="left_wheel"/>
-    <origin xyz="0 0.195 0" rpy="${-pi/2} 0 0"/>
+    <origin xyz="0 0.195 0" rpy="${-PI/2} 0 0"/>
     <axis xyz="0 0 1"/>
   </joint>
@@ -59,5 +59,5 @@
   <link name="right_wheel">
     <visual>
-      <origin xyz="0 0 0" rpy="0 ${-pi/2} 0"/>
+      <origin xyz="0 0 0" rpy="0 ${-PI/2} 0"/>
       <geometry>
         <mesh scale="1 1 1" filename="package://uiabot/urdf/meshes/wheel.stl"/>
@@ -77,5 +77,5 @@
   <!-- Robot base to right wheel joint -->
   <joint name="base_link_to_right_wheel" type="continuous">
-    <origin xyz="0 -0.195 0" rpy="${-pi/2} 0 0"/>
+    <origin xyz="0 -0.195 0" rpy="${-PI/2} 0 0"/>
     <parent link="base_link"/>
     <child link="right_wheel"/>
@@ -105,5 +105,5 @@
     <parent link="base_link"/>
     <child link="bno055"/>
-    <origin xyz="-0.2525 -0.117 0.0395" rpy="0 0 0"/>
+    <origin xyz="-0.305 0 0.0695" rpy="0 0 0"/>
   </joint>
   <!-- Lidar link -->
@@ -121,5 +121,5 @@
     <parent link="base_link"/>
     <child link="laser"/>
-    <origin xyz="-0.283 0.0 0.18" rpy="0 0 0"/>
+    <origin xyz="-0.278 0.0 0.18" rpy="0 0 0"/>
   </joint>
 </robot>

Commit message: temp updates

File: urdf/uiabot.urdf.xacro (robot description, xacro)
@@ -3,4 +3,12 @@
   <!-- Properties -->
   <xacro:property name="PI" value="3.1415926535897931"/>
+     <!-- Base footprint -->
+  <link name="base_footprint"/>
+  <!-- Base footprint to base link joint -->
+  <joint name="base_footprint_to_base_link" type="fixed">
+    <parent link="base_footprint"/>
+    <child link="base_link"/>
+    <origin xyz="0 0 0" rpy="0 0 0"/>
+  </joint>
   <!-- Robot base link-->
   <link name="base_link">
@@ -22,12 +30,4 @@
     </collision>
   </link>
-   <!-- Base footprint -->
-  <link name="base_footprint"/>
-  <!-- Base footprint to base link joint -->
-  <joint name="base_footprint_to_base_link" type="fixed">
-    <parent link="base_link"/>
-    <child link="base_footprint"/>
-    <origin xyz="0 0 0" rpy="0 0 0"/>
-  </joint>
   <!-- Left wheel link -->
   <link name="left_wheel">

Commit message: updated URDF

File: urdf/uiabot.urdf.xacro (robot description, xacro)
@@ -5,10 +5,4 @@
      <!-- Base footprint -->
   <link name="base_footprint"/>
-  <!-- Base footprint to base link joint -->
-  <joint name="base_footprint_to_base_link" type="fixed">
-    <parent link="base_footprint"/>
-    <child link="base_link"/>
-    <origin xyz="0 0 0" rpy="0 0 0"/>
-  </joint>
   <!-- Robot base link-->
   <link name="base_link">
@@ -30,4 +24,10 @@
     </collision>
   </link>
+    <!-- Base footprint to base link joint -->
+  <joint name="base_footprint_to_base_link" type="fixed">
+    <parent link="base_footprint"/>
+    <child link="base_link"/>
+    <origin xyz="0 0 0.055;" rpy="0 0 0"/>
+  </joint>
   <!-- Left wheel link -->
   <link name="left_wheel">
@@ -53,5 +53,5 @@
     <parent link="base_link"/>
     <child link="left_wheel"/>
-    <origin xyz="0 0.195 0" rpy="${-pi/2} 0 0"/>
+    <origin xyz="0.129 0.195 0" rpy="${-pi/2} 0 0"/>
     <axis xyz="0 0 1"/>
   </joint>
@@ -77,5 +77,5 @@
   <!-- Robot base to right wheel joint -->
   <joint name="base_link_to_right_wheel" type="continuous">
-    <origin xyz="0 -0.195 0" rpy="${-pi/2} 0 0"/>
+    <origin xyz="0.129 -0.195 0" rpy="${-pi/2} 0 0"/>
     <parent link="base_link"/>
     <child link="right_wheel"/>
@@ -105,5 +105,5 @@
     <parent link="base_link"/>
     <child link="bno055"/>
-    <origin xyz="-0.2525 -0.117 0.0395" rpy="0 0 0"/>
+    <origin xyz="-0.17 0.0 0.06" rpy="0 0 0"/>
   </joint>
   <!-- Lidar link -->
@@ -121,5 +121,5 @@
     <parent link="base_link"/>
     <child link="laser"/>
-    <origin xyz="-0.283 0.0 0.18" rpy="0 0 0"/>
+    <origin xyz="-0.14 0.0 0.18" rpy="0 0 0"/>
   </joint>
 </robot>

Commit message: fixed urdf

File: urdf/uiabot.urdf.xacro (robot description, xacro)
@@ -28,5 +28,5 @@
     <parent link="base_footprint"/>
     <child link="base_link"/>
-    <origin xyz="0 0 0.055;" rpy="0 0 0"/>
+    <origin xyz="0 0 0.055" rpy="0 0 0"/>
   </joint>
   <!-- Left wheel link -->

Commit message: Fixed corrupted stl files isssue

File: urdf/uiabot.urdf.xacro (robot description, xacro)
@@ -10,5 +10,5 @@
       <origin xyz="0.0 0.0 0.0" rpy="0 0 ${-PI/2}" />
       <geometry>
-        <mesh scale="1 1 1" filename="package://uiabot/urdf/meshes/uiabot.stl"/>
+        <mesh scale="1 1 1" filename="package://uiabot/urdf/meshes/uiabot.dae"/>
       </geometry>
       <material name="gray">
@@ -35,5 +35,5 @@
       <origin xyz="0 0 0" rpy="0 ${pi/2} 0" />
       <geometry>
-        <mesh scale="1 1 1" filename="package://uiabot/urdf/meshes/wheel.stl"/>
+        <cylinder radius="0.055" length="0.048" />
       </geometry>
       <material name="gray">
@@ -61,5 +61,5 @@
       <origin xyz="0 0 0" rpy="0 ${-pi/2} 0"/>
       <geometry>
-        <mesh scale="1 1 1" filename="package://uiabot/urdf/meshes/wheel.stl"/>
+        <cylinder radius="0.055" length="0.048" />
       </geometry>
       <material name="gray">
@@ -123,3 +123,28 @@
     <origin xyz="-0.14 0.0 0.18" rpy="0 0 0"/>
   </joint>
+  <!-- Caster wheel link -->
+  <link name="caster_wheel">
+    <visual>
+      <origin xyz="0 0 0" rpy="0 0 0" />
+      <geometry>
+        <sphere radius="0.02" />
+      </geometry>
+      <material name="gray">
+        <color rgba=".2 .2 .2 1" />
+      </material>
+    </visual>
+    <collision>
+      <origin xyz="0 0 0" rpy="0 0 0" />
+      <geometry>
+        <sphere radius="0.02" />
+      </geometry>
+      <contact_coefficients mu="0" kp="1000.0" kd="1.0"/>
+    </collision>
+  </link>
+  <!-- Caster wheel joint -->
+  <joint name="base_link_to_caster_wheel" type="fixed">
+    <parent link="base_link"/>
+    <child link="caster_wheel"/>
+    <origin xyz="-0.18 0.0 -0.035" rpy="0 0 0"/>
+  </joint>
 </robot>

Commit message: update URDF

File: urdf/uiabot.urdf.xacro (robot description, xacro)
@@ -42,5 +42,5 @@
     </visual>
     <collision>
-      <origin xyz="0 0 0" />
+      <origin xyz="0 0 0" rpy="0 ${pi/2} 0" />
       <geometry>
         <cylinder radius="0.055" length="0.048" />
@@ -53,5 +53,5 @@
     <parent link="base_link"/>
     <child link="left_wheel"/>
-    <origin xyz="0.129 0.195 0" rpy="${-pi/2} 0 0"/>
+    <origin xyz="0.0 0.195 0" rpy="${-pi/2} 0 0"/>
     <axis xyz="0 0 1"/>
   </joint>
@@ -59,5 +59,5 @@
   <link name="right_wheel">
     <visual>
-      <origin xyz="0 0 0" rpy="0 ${-pi/2} 0"/>
+      <origin xyz="0 0 0" rpy="0 ${pi/2} 0" />
       <geometry>
         <cylinder radius="0.055" length="0.048" />
@@ -68,5 +68,5 @@
     </visual>
     <collision>
-      <origin xyz="0 0 0" />
+      <origin xyz="0 0 0" rpy="0 ${pi/2} 0" />
       <geometry>
         <cylinder radius="0.055" length="0.048" />
@@ -77,5 +77,5 @@
   <!-- Robot base to right wheel joint -->
   <joint name="base_link_to_right_wheel" type="continuous">
-    <origin xyz="0.129 -0.195 0" rpy="${-pi/2} 0 0"/>
+    <origin xyz="0.0 -0.195 0" rpy="${-pi/2} 0 0"/>
     <parent link="base_link"/>
     <child link="right_wheel"/>
@@ -105,5 +105,5 @@
     <parent link="base_link"/>
     <child link="bno055"/>
-    <origin xyz="-0.17 0.0 0.06" rpy="0 0 0"/>
+    <origin xyz="-0.299 0.0 0.06" rpy="0 0 0"/>
   </joint>
   <!-- Lidar link -->
@@ -121,5 +121,5 @@
     <parent link="base_link"/>
     <child link="laser"/>
-    <origin xyz="-0.14 0.0 0.18" rpy="0 0 0"/>
+    <origin xyz="-0.269 0.0 0.18" rpy="0 0 0"/>
   </joint>
   <!-- Caster wheel link -->

Commit message: fixed URDF

File: urdf/uiabot.urdf.xacro (robot description, xacro)
@@ -28,10 +28,10 @@
     <parent link="base_footprint"/>
     <child link="base_link"/>
-    <origin xyz="0 0 0.055" rpy="0 0 0"/>
+    <origin xyz="0.129 0 0.055" rpy="0 0 0"/>
   </joint>
   <!-- Left wheel link -->
   <link name="left_wheel">
     <visual>
-      <origin xyz="0 0 0" rpy="0 ${pi/2} 0" />
+      <origin xyz="0 0 0" rpy="0 0 0" />
       <geometry>
         <cylinder radius="0.055" length="0.048" />
@@ -59,5 +59,5 @@
   <link name="right_wheel">
     <visual>
-      <origin xyz="0 0 0" rpy="0 ${pi/2} 0" />
+      <origin xyz="0 0 0" rpy="0 0 0" />
       <geometry>
         <cylinder radius="0.055" length="0.048" />
@@ -121,30 +121,5 @@
     <parent link="base_link"/>
     <child link="laser"/>
-    <origin xyz="-0.269 0.0 0.18" rpy="0 0 0"/>
-  </joint>
-  <!-- Caster wheel link -->
-  <link name="caster_wheel">
-    <visual>
-      <origin xyz="0 0 0" rpy="0 0 0" />
-      <geometry>
-        <sphere radius="0.02" />
-      </geometry>
-      <material name="gray">
-        <color rgba=".2 .2 .2 1" />
-      </material>
-    </visual>
-    <collision>
-      <origin xyz="0 0 0" rpy="0 0 0" />
-      <geometry>
-        <sphere radius="0.02" />
-      </geometry>
-      <contact_coefficients mu="0" kp="1000.0" kd="1.0"/>
-    </collision>
-  </link>
-  <!-- Caster wheel joint -->
-  <joint name="base_link_to_caster_wheel" type="fixed">
-    <parent link="base_link"/>
-    <child link="caster_wheel"/>
-    <origin xyz="-0.18 0.0 -0.035" rpy="0 0 0"/>
+    <origin xyz="-0.28 0.0 0.18" rpy="0 0 0"/>
   </joint>
 </robot>

Commit message: updated uiabot urdf

File: urdf/uiabot.urdf.xacro (robot description, xacro)
@@ -53,5 +53,5 @@
     <parent link="base_link"/>
     <child link="left_wheel"/>
-    <origin xyz="0.0 0.195 0" rpy="${-pi/2} 0 0"/>
+    <origin xyz="0.0 0.185 0" rpy="${-pi/2} 0 0"/>
     <axis xyz="0 0 1"/>
   </joint>
@@ -77,5 +77,5 @@
   <!-- Robot base to right wheel joint -->
   <joint name="base_link_to_right_wheel" type="continuous">
-    <origin xyz="0.0 -0.195 0" rpy="${-pi/2} 0 0"/>
+    <origin xyz="0.0 -0.185 0" rpy="${-pi/2} 0 0"/>
     <parent link="base_link"/>
     <child link="right_wheel"/>
